File: Speaker Amp/Speaker Amp.kicad_pcb (KiCad board)
At the start: 2 copper layers, 46.4 x 52.1 mm, 56 parts, among them J1 USB_C_Receptacle_USB2.0_16P, J2 Screw_Terminal_01x02, J3 Screw_Terminal_01x02, J4 Screw_Terminal_01x02, SW1 SW_Push, SW2 SW_Push, SW3 SW_Push, U1 LD1117S33TR_SOT223, U2 PCM2704CDBR, U3 TDA7297, U4 CH221K, Y1 12M

Commit message: Speaker Amp: swap 5.08mm Phoenix terminals to 3.5mm 4Ucon (Detkin stock)
In-place footprint swap for J2/J3/J4, pads recentered on the old blocks,
nets preserved, Phoenix PT-1,5 step model attached (no 4Ucon model ships).
Electrolytics already matched the user's THT caps. DRC unchanged: only the
accepted R6 starved-thermal.

Co-Authored-By: Claude Fable 5 <noreply@anthropic.com>
Parts:
- J2, J3, J4: footprint TerminalBlock_Phoenix:TerminalBlock_Phoenix_MKDS-1,5-2-5.08_1x02_P5.08mm_Horizontal -> TerminalBlock_4Ucon_1x02_P3.50mm_Horizontal
- moved J3 0.79 mm to (108.0, 52.5)
- moved J4 0.79 mm to (108.0, 75.4)
- moved J2 0.79 mm to (108.0, 64.0)

Commit message: Speaker Amp V4: JLC-mountable protection parts, THT indicator LED
- D2: P6KE16A DO-15 -> SMBJ15A SMB (JLC Preferred C19077569); schematic
  symbol rotated so the cathode pad lands on VBUS_RAW for assembly polarity
- F1: Bourns MF-RG300 radial -> SMD1812P300TF/16 3A/16V 1812 (C702820);
  C_1812 chip step model as stand-in (no 1812 fuse model ships)
- D1: APA1606 side LED -> LED_THT:LED_D5.0mm (Detkin stock, matches visualizer)
- User rework of the power-entry routing; one missing VBUS_RAW F/B via
  restored where the old D2 through-hole used to bridge layers
- DRC: 0 violations except accepted R6 starved-thermal, 0 unconnected
- V4 render set

Co-Authored-By: Claude Fable 5 <noreply@anthropic.com>
Parts:
- D1: footprint LED_SMD:LED_Kingbright_APA1606_1.6x0.6mm_Horizontal -> LED_D5.0mm
- D2: footprint Diode_THT:D_DO-15_P10.16mm_Horizontal -> D_SMB
- F1: footprint Fuse:Fuse_Bourns_MF-RG300 -> Fuse_1812_4532Metric
- moved REF** 12.1 mm to (99.1, 68.6)
- moved J4 6.83 mm to (107.7, 68.6)
- moved J2 4.30 mm to (107.7, 59.7)
- moved REF** 3.17 mm to (110.5, 31.8)
- moved REF** 3.17 mm to (71.1, 31.8)
- moved F1 2.62 mm to (81.3, 42.6)
- moved D1 2.54 mm to (71.1, 39.4)
- moved D2 2.19 mm to (76.8, 37.1), turned to 90 degrees
- moved J3 1.77 mm to (107.7, 50.8)
Connections:
- D2 pad 1: GND -> /VBUS_RAW
- D2 pad 2: /VBUS_RAW -> GND
Routing:
- net /+12V: track 109.2 -> 98.1 mm
- net /VBUS_RAW: track 19.8 -> 29.4 mm, vias 1 -> 2
- net Net-(D1-K): track 24.0 -> 20.6 mm, vias 0 -> 1
- net /OUT_L+: track 7.25 -> 8.59 mm
- net /OUT_R+: track 9.88 -> 8.59 mm
- net GND: track 50.1 -> 51.1 mm, vias 26 -> 28
- net /OUT_L-: track 23.5 -> 22.8 mm
- net /OUT_R-: track 14.8 -> 14.2 mm
Other:
- board size 46.4 x 52.1 mm -> 46.4 x 55.2 mm

Commit message: Regenerate JLCPCB fab packages: Visualizer V2, Speaker Amp V4
Fresh gerbers/drill, BOM and CPL from the current boards, updated READMEs.
Both DRC-clean with 0 unconnected and 0 schematic parity issues. D2 board
value synced to SMBJ15A. Versioned zips are local-only (gitignored).

Co-Authored-By: Claude Fable 5 <noreply@anthropic.com>
Parts:
- D2: value P6KE16A -> SMBJ15A
Changed lines of the file:
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@@
 			)
 		)
-		(property "Value" "P6KE16A"
+		(property "Value" "SMBJ15A"
 			(at 0 3.1 90)
 			(layer "F.Fab")

Commit message: Speaker Amp: Basic-catalog U1/Y1, fab package refresh
- U1: LD1117S33 -> AMS1117-3.3 (C6186, Basic, pin-compatible SOT-223)
- Y1: explicit LCSC C9002 (12MHz 3225, Basic) so the matcher stops
  whiffing on the custom 2-pin-remapped footprint name
- D2 C19077569 confirmed on JLC's Preferred list (no fee despite the
  Extended label in the matcher UI)
- Remaining fee-carrying Extended: F1, J1, SW1-3, U2, U4 (+U3 unless DNP)

Co-Authored-By: Claude Fable 5 <noreply@anthropic.com>
Parts:
- U1: value LD1117S33TR_SOT223 -> AMS1117-3.3
Changed lines of the file:
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@@
 			)
 		)
-		(property "Value" "LD1117S33TR_SOT223"
+		(property "Value" "AMS1117-3.3"
 			(at 0 4.5 90)
 			(layer "F.Fab")
