File: Audio Visualizer/Audio Visualizer.kicad_pcb (KiCad board)
At the start: 2 copper layers, 106.7 x 29.8 mm, 122 parts, among them J3 Screw_Terminal_01x02, J4 Screw_Terminal_01x02, J5 Screw_Terminal_01x02, J6 Screw_Terminal_01x02, J7 Screw_Terminal_01x02, Q10 MMBT3904, Q11 MMBT3904, Q12 MMBT3904, Q13 MMBT3904, Q14 MMBT3904, Q15 MMBT3904, Q16 MMBT3904, Q17 MMBT3904, Q18 MMBT3904, Q19 MMBT3904, Q2 MMBT3904, Q20 MMBT3904, Q21 MMBT3904, Q3 MMBT3904, Q4 MMBT3904, Q5 MMBT3904, Q6 MMBT3904, Q7 MMBT3904, Q8 MMBT3904, Q9 MMBT3904, U1 LM358

Commit message: Audio Visualizer: all-Basic resistor ladder (free Rtop/Rk pairs)
Ladder recalculated per stage from JLC's Basic 0805 catalog with both
divider resistors free; same -22.5..0dB / 2.5dB thresholds. Worst error
improves 3.8% -> 1.4%; op-amp load drops ~9.9 -> ~6.5mA per channel.
Gain 2.1 rebuilt as 1 + 22k/20k (11k was Extended). 36 value changes in
sch + PCB, no layout changes. Docs updated (user), fab package folders
restructured to JLCPCB_*_V2/V4 and visualizer package regenerated.

Co-Authored-By: Claude Fable 5 <noreply@anthropic.com>
Parts:
- R10, R22, R43, R55: value 10k -> 27k
- R11, R44: value 9.1k -> 24k
- R13, R25, R46, R58: value 10k -> 22k
- R14, R47: value 5.1k -> 12k
- R16, R49: value 10k -> 6.8k
- R17, R50: value 3.6k -> 2.4k
- R23, R56: value 1.8k -> 4.7k
- R26, R59: value 1.2k -> 2.7k
- R28, R61: value 10k -> 30k
- R29, R62: value 910 -> 2.7k
- R31, R64: value 10k -> 15k
- R32, R65: value 680 -> 1k
- R35, R40, R6, R7: value 10k -> 20k
- R36, R5: value 11k -> 22k
- R41, R8: value 16k -> 33k
Changed lines of the file:
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@@
 			)
 		)
-		(property "Value" "910"
+		(property "Value" "2.7k"
 			(at 0 1.65 90)
 			(layer "F.Fab")
@@
 			)
 		)
-		(property "Value" "10k"
+		(property "Value" "6.8k"
 			(at 0 1.65 90)
 			(layer "F.Fab")
@@
 			)
 		)
-		(property "Value" "11k"
+		(property "Value" "22k"
 			(at 0 1.65 90)
 			(layer "F.Fab")
@@
 			)
 		)
-		(property "Value" "3.6k"
+		(property "Value" "2.4k"
 			(at 0 1.65 90)
 			(layer "F.Fab")
@@
 			)
 		)
-		(property "Value" "10k"
+		(property "Value" "30k"
 			(at 0 1.65 90)
 			(layer "F.Fab")
@@
 			)
 		)
-		(property "Value" "10k"
+		(property "Value" "6.8k"
 			(at 0 1.65 90)
 			(layer "F.Fab")
@@
 			)
 		)
-		(property "Value" "10k"
+		(property "Value" "15k"
 			(at 0 1.65 90)
 			(layer "F.Fab")
@@
 			)
 		)
-		(property "Value" "9.1k"
+		(property "Value" "24k"
 			(at 0 1.65 90)
 			(layer "F.Fab")
@@
 			)
 		)
-		(property "Value" "9.1k"
+		(property "Value" "24k"
 			(at 0 1.65 90)
 			(layer "F.Fab")
@@
 			)
 		)
-		(property "Value" "10k"
+		(property "Value" "27k"
 			(at 0 1.65 90)
 			(layer "F.Fab")
@@
 			)
 		)
-		(property "Value" "10k"
+		(property "Value" "20k"
 			(at 0 1.65 90)
 			(layer "F.Fab")
@@
 			)
 		)
-		(property "Value" "10k"
+		(property "Value" "15k"
 			(at 0 1.65 90)
 			(layer "F.Fab")
@@
 			)
 		)
-		(property "Value" "10k"
+		(property "Value" "27k"
 			(at 0 1.65 90)
 			(layer "F.Fab")
@@
 			)
 		)
-		(property "Value" "1.2k"
+		(property "Value" "2.7k"
 			(at 0 1.65 90)
 			(layer "F.Fab")
@@
 			)
 		)
-		(property "Value" "10k"
+		(property "Value" "20k"
 			(at 0 1.65 0)
 			(layer "F.Fab")
@@
 			)
 		)
-		(property "Value" "1.8k"
+		(property "Value" "4.7k"
 			(at 0 1.65 90)
 			(layer "F.Fab")
@@
 			)
 		)
-		(property "Value" "11k"
+		(property "Value" "22k"
 			(at 0 1.65 90)
 			(layer "F.Fab")
@@
 			)
 		)
-		(property "Value" "10k"
+		(property "Value" "22k"
 			(at 0 1.65 90)
 			(layer "F.Fab")
@@
 			)
 		)
-		(property "Value" "5.1k"
+		(property "Value" "12k"
 			(at 0 1.65 90)
 			(layer "F.Fab")
@@
 			)
 		)
-		(property "Value" "680"
+		(property "Value" "1k"
 			(at 0 1.65 90)
 			(layer "F.Fab")
@@
 			)
 		)
-		(property "Value" "16k"
+		(property "Value" "33k"
 			(at 0 1.65 90)
 			(layer "F.Fab")
@@
 			)
 		)
-		(property "Value" "10k"
+		(property "Value" "27k"
 			(at 0 1.65 90)
 			(layer "F.Fab")
@@
 			)
 		)
-		(property "Value" "10k"
+		(property "Value" "22k"
 			(at 0 1.65 90)
 			(layer "F.Fab")
@@
 			)
 		)
-		(property "Value" "3.6k"
+		(property "Value" "2.4k"
 			(at 0 1.65 90)
 			(layer "F.Fab")
@@
 			)
 		)
-		(property "Value" "10k"
+		(property "Value" "22k"
 			(at 0 1.65 90)
 			(layer "F.Fab")
@@
 			)
 		)
-		(property "Value" "5.1k"
+		(property "Value" "12k"
 			(at 0 1.65 90)
 			(layer "F.Fab")
@@
 			)
 		)
-		(property "Value" "680"
+		(property "Value" "1k"
 			(at 0 1.65 90)
 			(layer "F.Fab")
@@
 			)
 		)
-		(property "Value" "10k"
+		(property "Value" "20k"
 			(at 0 1.65 0)
 			(layer "F.Fab")
@@
 			)
 		)
-		(property "Value" "10k"
+		(property "Value" "30k"
 			(at 0 1.65 90)
 			(layer "F.Fab")
@@
 			)
 		)
-		(property "Value" "1.8k"
+		(property "Value" "4.7k"
 			(at 0 1.65 90)
 			(layer "F.Fab")
@@
 			)
 		)
-		(property "Value" "10k"
+		(property "Value" "20k"
 			(at 0 1.65 90)
 			(layer "F.Fab")
@@
 			)
 		)
-		(property "Value" "910"
+		(property "Value" "2.7k"
 			(at 0 1.65 90)
 			(layer "F.Fab")
@@
 			)
 		)
-		(property "Value" "16k"
+		(property "Value" "33k"
 			(at 0 1.65 90)
 			(layer "F.Fab")
@@
 			)
 		)
-		(property "Value" "10k"
+		(property "Value" "22k"
 			(at 0 1.65 90)
 			(layer "F.Fab")
@@
 			)
 		)
-		(property "Value" "1.2k"
+		(property "Value" "2.7k"
 			(at 0 1.65 90)
 			(layer "F.Fab")
@@
 			)
 		)
-		(property "Value" "10k"
+		(property "Value" "27k"
 			(at 0 1.65 90)
 			(layer "F.Fab")

Commit message: Terminals flipped to face outward (user rework), renders/STEPs regenerated
User rotated and repositioned all eight screw terminals so wire entries
face the board edges; copper reworked accordingly, DRC/parity clean on
both boards. All render sets, layout PNGs, and STEP files regenerated.

Co-Authored-By: Claude Fable 5 <noreply@anthropic.com>
Parts:
- moved J4 3.50 mm to (100.5, 110.0), turned to 0 degrees
- moved J5 3.50 mm to (90.5, 110.0), turned to 0 degrees
- moved J6 3.50 mm to (93.5, 88.5), turned to 180 degrees
- moved J7 3.50 mm to (103.5, 88.5), turned to 180 degrees
- moved J3 3.46 mm to (91.2, 97.8), turned to -90 degrees
Routing:
- net /IN_R+: track 17.9 -> 15.9 mm
- net /+12V: track 388.7 -> 387.7 mm
