File: Audio Visualizer/Audio Visualizer.kicad_pcb (KiCad board)
At the start: 2 copper layers, 106.7 x 29.8 mm, 122 parts, among them J3 Screw_Terminal_01x02, J4 Screw_Terminal_01x02, J5 Screw_Terminal_01x02, J6 Screw_Terminal_01x02, J7 Screw_Terminal_01x02, Q10 MMBT3904, Q11 MMBT3904, Q12 MMBT3904, Q13 MMBT3904, Q14 MMBT3904, Q15 MMBT3904, Q16 MMBT3904, Q17 MMBT3904, Q18 MMBT3904, Q19 MMBT3904, Q2 MMBT3904, Q20 MMBT3904, Q21 MMBT3904, Q3 MMBT3904, Q4 MMBT3904, Q5 MMBT3904, Q6 MMBT3904, Q7 MMBT3904, Q8 MMBT3904, Q9 MMBT3904, U1 LM358

Commit message: Audio Visualizer: mount screw terminals J3-J7 on underside
Flipped the five 3.5mm terminal blocks to B.Cu so the LED/top face sits
flush (e.g. against the front panel), wires now enter from the back into
the enclosure. THT holes and nets unchanged -> traces untouched, schematic
parity clean, DRC 0/0. Renders, layout, and STEP regenerated.

NOTE: diverges from the already-ordered boards (terminals top-side); this
is next-rev / enclosure-design geometry. Fab packages intentionally NOT
regenerated.

Co-Authored-By: Claude Opus 4.8 <noreply@anthropic.com>
Parts:
- J3, J4, J5, J6, J7: moved to B.Cu

Commit message: Audio Visualizer: move C2/C4 10uF electrolytics to underside too
Flipped the two THT radials to B.Cu alongside the terminals so the top
face carries only the LED ladder + SMD parts (maximally flush). Polarity
preserved (parity clean), holes/nets unchanged, DRC 0/0/0, no courtyard
collisions with the bottom-side terminals. Renders + STEP regenerated.

Co-Authored-By: Claude Opus 4.8 <noreply@anthropic.com>
Parts:
- C2, C4: moved to B.Cu
